Commit message: Week 5: fix(pr-d): resolve Gazebo Ignition launch issues, update README
- Wrap robot_description/SRDF with ParameterValue(value_type=str)
- Add <link name='world'/> for ur_description base_joint
- Use ign_ros2_control plugin naming for Humble+Fortress
- Simplify gz_bridge to arguments-based config
- Set IGN_GAZEBO_SYSTEM_PLUGIN_PATH=/opt/ros/humble/lib
- Add comprehensive Quick Start, deps, and Troubleshooting to README
- Clean unused imports in launch files

File: enfield_robots_ur5e/urdf/ur5e_enfield.urdf.xacro (robot description, xacro)
@@ -27,4 +27,6 @@
   <!-- ============================================================ -->
   <xacro:include filename="$(find ur_description)/urdf/ur_macro.xacro"/>
+  <!-- World link required by ur_description base_joint -->
+  <link name="world"/>
   <!-- ============================================================ -->
   <!-- Instantiate the UR5e robot                                    -->
@@ -51,6 +53,6 @@
   <xacro:if value="$(arg sim_ignition)">
     <gazebo>
-      <plugin filename="gz_ros2_control-system"
-              name="gz_ros2_control::GazeboSimROS2ControlPlugin">
+      <plugin filename="ign_ros2_control-system"
+              name="ign_ros2_control::IgnitionROS2ControlPlugin">
         <parameters>$(find enfield_robots_ur5e)/config/ur5e_controllers.yaml</parameters>
       </plugin>
